File: cbm2ram.sch (EAGLE design)
At the start: 21 parts, among them U1 74574N, U2 74574N, U3 GAL16V8, U4 74LS04N, U5 HM628512A_DIL32, U6 HM628512A_DIL32, U7 74541N, U8 74541N

Commit message: Added EPROM chips
Parts:
- added C10, C11, C12, C9: 330n, capacitor-wima:C5/3
- added U10, U11, U12: 27C64P, microchip:27C64P
- added U9: 74138N, 74ttl-din@1:74138N
Connections:
- new net /WE: CONN3.19, U10.PGM, U11.PGM, U12.PGM, U4D.I
- new net MD0: CONN3.36, U10.D0, U11.D0, U12.D0
- new net MD1: CONN3.34, U10.D1, U11.D1, U12.D1
- new net MD2: CONN3.32, U10.D2, U11.D2, U12.D2
- new net MD3: CONN3.29, U10.D3, U11.D3, U12.D3
- new net MD4: CONN3.31, U10.D4, U11.D4, U12.D4
- new net MD5: CONN3.33, U10.D5, U11.D5, U12.D5
- new net MD6: CONN3.35, U10.D6, U11.D6, U12.D6
- new net MD7: CONN3.38, U10.D7, U11.D7, U12.D7
- new net N$2: U12.!CE, U91.Y3
- new net N$3: U11.!CE, U91.Y2
- new net N$5: U10.!CE, U91.Y1
- new net N$8: U10.!OE, U11.!OE, U12.!OE, U4D.O
- net A0: now also U10.A0, U11.A0, U12.A0
- net A1: now also U10.A1, U11.A1, U12.A1
- net A10: now also U10.A10, U11.A10, U12.A10
- net A11: now also U10.A11, U11.A11, U12.A11
- net A12: now also U10.A12, U11.A12, U12.A12
- net A13: now also U91.A
- net A14: now also U91.B
- net A15: now also U91.C
- net A2: now also U10.A2, U11.A2, U12.A2
- net A3: now also U10.A3, U11.A3, U12.A3
- net A4: now also U10.A4, U11.A4, U12.A4
- net A5: now also U10.A5, U11.A5, U12.A5
- net A6: now also U10.A6, U11.A6, U12.A6
- net A7: now also U10.A7, U11.A7, U12.A7
- net A8: now also U10.A8, U11.A8, U12.A8
- net A9: now also U10.A9, U11.A9, U12.A9
- net BANK15: now also U91.!G2A, U91.!G2B
- net GND: now also C10.1, C11.1, C12.1, C9.1, U10.GND, U11.GND, U12.GND, U9/-UB.-UB
- net VCC: now also C10.2, C11.2, C12.2, C9.2, U10.VCC, U10.VPP, U11.VCC, U11.VPP, U12.VCC, U12.VPP, U9/+UB.+UB, U91.G1
Other:
- moved on the sheet: C1, C2, C3, C4, C5, C6, C7, C8

Commit message: Complete board.
Parts:
- removed JP1: (no value), jumper:JP1E
- added C13: 220n, capacitor-wima:C5/3
- R1: value 5.1k -> 1k
- U10, U11, U12: value 27C64P -> (none); device microchip:27C64P -> memory-hitachi:6264A
- U3: value GAL16V8 -> (none); device pal:16V8 -> pal:22V10
- U9: value 74138N -> (none); device 74ttl-din@1:74138N -> memory-hitachi:6264A
Connections:
- removed net /P2REFGNT: CONN1.26, CONN2.26
- removed net /WE: CONN3.19, U10.PGM, U11.PGM, U12.PGM, U4D.I
- removed net BANK15: U3G$1.O7, U91.!G2A, U91.!G2B
- removed net N$1: JP1.1, R1.1, U3G$1.I6
- removed net N$2: U12.!CE, U91.Y3
- removed net N$3: U11.!CE, U91.Y2
- removed net N$5: U10.!CE, U91.Y1
- removed net N$8: U10.!OE, U11.!OE, U12.!OE, U4D.O
- new net /ECAS': U3G$1.I10, U4E.O
- new net /OE: U10.!OE, U11.!OE, U12.!OE, U4D.O, U9.!OE
- new net /RAM1: U12.!CS1, U3G$1.O6
- new net /ROM1: U3G$1.O7, U9.!CS1
- new net /ROM2: U10.!CS1, U3G$1.O8
- new net /ROM3: U11.!CS1, U3G$1.O9
- new net ECAS': C13.1, R1.1, U4E.I
- new net PHI1: CONN3.27, U3G$1.I3
- net /BUSY2: now also U3G$1.I9; no longer U3G$1.I5
- net /CAS: now also CONN1.26, U3G$1.I8; no longer U3G$1.I4
- net /CS1: now also U3G$1.O1; no longer U3G$1.O5
- net /CS2: now also U3G$1.O0; no longer U3G$1.O6
- net /ECAS: no longer CONN1.40, U3G$1.I7
- net /ERAS: no longer CONN1.38
- net A0: now also U9.A0
- net A1: now also U9.A1
- net A10: now also U9.A10
- net A11: now also U9.A11
- net A12: now also U3G$1.CLK/I0, U9.A12
- net A13: now also U3G$1.I0; no longer U91.A
- net A14: now also U3G$1.I1; no longer U91.B
- net A15: now also U3G$1.I2; no longer U91.C
- net A2: now also U9.A2
- net A3: now also U9.A3
- net A4: now also U9.A4
- net A5: now also U9.A5
- net A6: now also U9.A6
- net A7: now also U9.A7
- net A8: now also U9.A8
- net A9: now also U9.A9
- net BP0: now also U3G$1.I4; no longer U3G$1.I0
- net BP1: now also U3G$1.I5; no longer U3G$1.I1
- net BP2: now also U3G$1.I6; no longer U3G$1.I2
- net BP3: now also U3G$1.I7; no longer U3G$1.I3
- net ECAS: now also R1.2, U21.CLK; no longer U11.CLK
- net ERAS: now also U11.CLK; no longer U21.CLK
- net GND: now also C13.2, U10.VSS, U11.VSS, U12.VSS, U9.VSS; no longer JP1.2, U10.GND, U11.GND, U12.GND, U9/-UB.-UB
- net MD0: now also U10.I/O1, U11.I/O1, U12.I/O1, U9.I/O1; no longer U10.D0, U11.D0, U12.D0
- net MD1: now also U10.I/O2, U11.I/O2, U12.I/O2, U9.I/O2; no longer U10.D1, U11.D1, U12.D1
- net MD2: now also U10.I/O3, U11.I/O3, U12.I/O3, U9.I/O3; no longer U10.D2, U11.D2, U12.D2
- net MD3: now also U10.I/O4, U11.I/O4, U12.I/O4, U9.I/O4; no longer U10.D3, U11.D3, U12.D3
- net MD4: now also U10.I/O5, U11.I/O5, U12.I/O5, U9.I/O5; no longer U10.D4, U11.D4, U12.D4
- net MD5: now also U10.I/O6, U11.I/O6, U12.I/O6, U9.I/O6; no longer U10.D5, U11.D5, U12.D5
- net MD6: now also U10.I/O7, U11.I/O7, U12.I/O7, U9.I/O7; no longer U10.D6, U11.D6, U12.D6
- net MD7: now also U10.I/O8, U11.I/O8, U12.I/O8, U9.I/O8; no longer U10.D7, U11.D7, U12.D7
- net R/W: now also U10.!WE, U11.!WE, U12.!WE, U4D.I, U9.!WE
- net VCC: now also CONN1.38, CONN1.40, U10.CS2, U11.CS2, U12.CS2, U9.CS2, U9.VCC; no longer R1.2, U10.VPP, U11.VPP, U12.VPP, U9/+UB.+UB, U91.G1
Other:
- moved on the sheet: CONN3, R1, U1/+UB, U4A, U4B, U4C, U4D, U5, U6, U7, U7/+UB, U7/-UB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
